File: pcb/Waberinator_hw2.kicad_sch (KiCad schematic)
At the start: 53 parts, among them J1 Power_UART, J10 Strang 5, J2 USB_OTG, J3 ISP, J4 Button, J5 Strang 0, J6 Strang 1, J7 Strang 2, J8 Strang 3, J9 Strang 4, Q1 SiZ340DT, Q2 SiZ340DT, U1 L7805, U2 ATMEGA8-16PU, U5 LM75B

Commit message: prepared for stm32f030. Assigned pins for timers and adcs. Selected mosfets and drivers
Parts:
- removed C1, C11, C3, C6: 100nF, symbol Waberinator_rev1-rescue:C
- removed C12: 2n, symbol Waberinator_rev1-rescue:C
- removed C13, C18: C, symbol Device:C
- removed C14: 22u, symbol Waberinator_rev1-rescue:C
- removed C15, C16: 1000u, symbol Waberinator_rev1-rescue:CP
- removed C2, C4: 22u, Capacitor_SMD:C_1206_3216Metric_Pad1.42x1.75mm_HandSolder, symbol Waberinator_rev1-rescue:C
- removed C7: ~, symbol Waberinator_rev1-rescue:CP
- removed C8: ~, symbol Waberinator_rev1-rescue:C
- removed D1: D_Schottky, Diode_THT:D_5W_P5.08mm_Vertical_AnodeUp, symbol Waberinator_rev1-rescue:D_Schottky
- removed D2: Red, symbol Waberinator_rev1-rescue:LED
- removed D3: Yellow, symbol Waberinator_rev1-rescue:LED
- removed D4: Green, symbol Waberinator_rev1-rescue:LED
- removed D5: SK34-TP, Diode_SMD:D_SMC_Handsoldering, symbol Device:D_Schottky
- removed J1: Power_UART, Connector_JST:JST_XH_B04B-XH-A_1x04_P2.50mm_Vertical, symbol Waberinator_rev1-rescue:Conn_01x04
- removed J10: Strang 5, symbol Connector_Generic:Conn_01x02
- removed J2: USB_OTG, Connector_USB:USB_Micro-B_Molex-105017-0001, symbol Waberinator_rev1-rescue:USB_OTG
- removed J3: ISP, Connector_Molex:Molex_Mega-Fit_76829-0110_2x05_P5.70mm_Vertical, symbol Waberinator_rev1-rescue:Conn_02x05_Odd_Even
- removed J4: Button, Connector_JST:JST_XH_B02B-XH-A_1x02_P2.50mm_Vertical, symbol Waberinator_rev1-rescue:Conn_01x02
- removed J8: Strang 3, symbol Connector_Generic:Conn_01x02
- removed J9: Strang 4, symbol Connector_Generic:Conn_01x02
- removed L1: 744770147, symbol Device:L
- removed Q1, Q2: SiZ340DT, g7_transistor:PowerPAIR3x3, symbol g7_transistor:DMG9926UDM
- removed R1: 10k, symbol Waberinator_rev1-rescue:R
- removed R2: 100, Resistor_SMD:R_0603_1608Metric_Pad1.05x0.95mm_HandSolder, symbol Waberinator_rev1-rescue:R
- removed R3: 270, symbol Waberinator_rev1-rescue:R
- removed R4: 200, symbol Waberinator_rev1-rescue:R
- removed R5: 360, symbol Waberinator_rev1-rescue:R
- removed R8: ~, symbol Waberinator_rev1-rescue:R
- removed R9: tbd, symbol Waberinator_rev1-rescue:R
- removed U1: L7805, Package_TO_SOT_THT:TO-220F-3_Horizontal_TabDown, symbol Waberinator_rev1-rescue:L7805
- removed U2: ATMEGA8-16PU, Package_DIP:DIP-28_W7.62mm_Socket_LongPads, symbol Waberinator_rev1-rescue:ATMEGA8-16PU
- removed U4: ~, symbol Regulator_Switching:LM2596S-ADJ
- removed U6, U7: ~, Package_DFN_QFN:DFN-8-1EP_3x3mm_P0.5mm_EP1.65x2.38mm, symbol g7_driver:ncp81155
- added C1: 479nF, symbol Device:C
- added C10: 100nF, Capacitor_SMD:C_0603_1608Metric_Pad1.08x0.95mm_HandSolder, symbol Waberinator_rev1-rescue:C
- added C16: 10n, symbol Waberinator_rev1-rescue:C
- added C21: 22µF, Capacitor_THT:C_Radial_D5.0mm_H11.0mm_P2.00mm, symbol Waberinator_rev1-rescue:CP
- added C3: 6.8pF, symbol Device:C
- added C5, C7: ~, Capacitor_SMD:C_0603_1608Metric_Pad1.08x0.95mm_HandSolder, symbol Device:C_Small
- added C5: 2.2µF, symbol Device:C
- added C9: 100nF, symbol Waberinator_rev1-rescue:C
- added D1: 824501121, Diode_SMD:D_SOD-128, symbol Device:D_TVS
- added D2: SD103CW-E3-08, Diode_SMD:D_SOD-123, symbol Device:D_Schottky
- added D3, D4, D5, D6: LED, symbol Device:LED
- added F1: ~, Fuse:Fuse_2512_6332Metric_Pad1.52x3.35mm_HandSolder, symbol Device:Fuse
- added FL1: ~, g7_emi:CMC_Laird_CM2021Y330R-10, symbol Device:EMI_Filter_LL_1423
- added J1: 12VDC In, Connector_JST:JST_XH_B2B-XH-A_1x02_P2.50mm_Vertical, symbol Connector:Conn_01x02_Pin
- added J11: Strang 0, symbol Connector:Conn_01x02_Male
- added J2: Strang 2, symbol Connector_Generic:Conn_01x02
- added J3: Strang 1, symbol Connector_Generic:Conn_01x02
- added J4: Strang 3, symbol Connector_Generic:Conn_01x02
- added L1: SRU1048-4R7Y, Inductor_SMD:L_Bourns_SRP1038C_10.0x10.0mm, symbol Device:L_Ferrite
- added NT1, NT2: NetTie_2, NetTie:NetTie-2_SMD_Pad0.5mm, symbol Device:NetTie_2
- added Q1: AOSP21321, Package_SO:SO-8_3.9x4.9mm_P1.27mm, symbol Device:Q_PMOS_DGS
- added Q2, Q3, Q4, Q5, Q6, Q7: SISHA04DN-T1-GE3, symbol Device:Q_NMOS_GDS
- added R1, R10, R3: 100k, symbol Device:R
- added R10, R8: 100, Resistor_SMD:R_0603_1608Metric_Pad0.98x0.95mm_HandSolder, symbol Device:R
- added R11, R12, R13, R14, R15, R2: 1, symbol Device:R
- added R16, R17, R18, R19: R, symbol Device:R
- added R4: 14.3k, symbol Device:R
- added R5: 117k, symbol Device:R
- added R9: 100k, Resistor_SMD:R_0603_1608Metric_Pad0.98x0.95mm_HandSolder, symbol Device:R
- added RV3: Brightness, g7_hmi:potentiometer_P160, symbol Waberinator_rev1-rescue:POT
- added SW1, SW2: SW_SPST, symbol Switch:SW_SPST
- added U2: LM73606QRNPRQ1, g7_ic:30-WFQFN-RNP0030A, symbol 2023-12-28_21-15-04:LM73606QRNPRQ1
- added U3: AMS1117-3.3, Package_TO_SOT_SMD:SOT-223-3_TabPin2, symbol Regulator_Linear:AMS1117-3.3
- added U3, U4, U6: MCP14A0304xMNY, Package_SO:SOIC-8_3.9x4.9mm_P1.27mm, symbol Driver_FET:MCP14A0304xMNY
- added U7: STM32F030R8Tx, Package_QFP:LQFP-64_10x10mm_P0.5mm, symbol MCU_ST_STM32F0:STM32F030R8Tx
- C17, C19: value C -> 100nF
- J5: value Strang 0 -> Strang 4
- J6: value Strang 1 -> Strang 5; Digikey (none) -> 609-3819-ND; MPN (none) -> OQ0232510000G
- J7: value Strang 2 -> Strang 6; Digikey (none) -> 609-3819-ND; MPN (none) -> OQ0232510000G
- R6: footprint (none) -> Resistor_SMD:R_0603_1608Metric_Pad0.98x0.95mm_HandSolder
- R7: value 33k -> 24,9k; footprint (none) -> Resistor_SMD:R_0603_1608Metric_Pad0.98x0.95mm_HandSolder
- RV1, RV2: footprint Potentiometer_THT:Potentiometer_Alps_RK097_Single_Horizontal -> g7_hmi:potentiometer_P160
- renumbered C9 to C14, C10 to C15
Connections:
- net +5V is gone; now on net +3.3V: RV1.1, RV2.1
- net +3.3V: now also RV3.1; no longer U5.8 (VCC)
- net adc_depth: now also U7.16 (PA2)
- net adc_frequency: now also U7.15 (PA1)
- net GND renamed RET
- net RET: now also C17.2, C19.2, C10.2, C16.2, C21.2, C5.2, C7.2, C9.2, D1.2 (A2), D2.2 (A), D3.1 (K), D4.1 (K), D5.1 (K), D6.1 (K), FL1.3, Q2.3 (S), Q3.3 (S), Q4.3 (S), Q5.3 (S), Q6.3 (S), Q7.3 (S), R10.2, R10.2, R4.2, R5.1, RV3.3, SW1.2 (B), SW2.2 (B), U2.12 (NC), U2.13 (NC), U2.14 (NC), U2.15 (NC), U2.17 (SYNC), U2.19 (AGND), U2.23 (PGND), U2.24 (PGND), U2.25 (PGND), U2.26 (PGND), U2.27 (NC), U2.28 (NC), U2.29 (NC), U2.30 (NC), U2.31 (DAP), U3.1 (GND), U3.3 (GND), U3.9 (GND), U4.3 (GND), U4.9 (GND), U6.3 (GND), U6.9 (GND), U7.12 (VSSA), U7.31 (VSS), U7.63 (VSS)
- net Vbat: no longer names the net of R6.2
- net Vbat: now also NT1.1
- net adc_vbat: no longer names the net of R6.1, R7.2
- net adc_vbat: now also C10.1, D2.1 (K), R8.1
- net bst1 renamed DC_prot
- net DC_prot: now also Q1.1 (S), Q1.2 (S), Q1.3 (S), U2.20 (VIN), U2.21 (VIN), U2.22 (VIN), U3.3 (VI)
- net bst2 renamed +3V3
- net +3V3: now also U5.8 (VCC), C21.1, C9.1, U3.2 (VO), U7.1 (VDD)
- net sw1 renamed VLed
- net VLed: now also C3.1, J2.1 (Pin_1), J3.1 (Pin_1), J4.1 (Pin_1), L1.2, R3.1, U2.8 (BIAS), U3.6 (V+), U4.6 (V+), U6.6 (V+); no longer C17.2
- removed net sw2: C19.2, J5.2 (Pin_2), J6.2 (Pin_2), J7.2 (Pin_2)
- new net: C3.2, R3.2, R4.1, U2.11 (FB)
- new net: J4.2 (Pin_2), Q4.2 (D)
- new net: J6.2 (Pin_2), Q6.2 (D)
- new net: R13.1, U4.5 (OUTB)
- new net: R12.1, U4.7 (OUTA)
- new net: Q5.1 (G), R13.2
- new net: J5.2 (Pin_2), Q5.2 (D)
- new net: D5.2 (A), R17.2
- new net: R5.2, U2.9 (RT)
- new net: J7.2 (Pin_2), Q7.2 (D)
- new net: NT2.1, R9.1
- new net: Q1.4 (G), R10.1, R9.2
- new net: R15.1, U6.5 (OUTB)
- new net: Q7.1 (G), R15.2
- new net: Q4.1 (G), R12.2
- new net: D4.2 (A), R18.2
- new net: J3.2 (Pin_2), Q3.2 (D)
- new net: R14.1, U6.7 (OUTA)
- new net: R2.1, U3.5 (OUTB)
- new net: Q2.1 (G), R2.2
- new net: C1.2, L1.1, U2.1 (SW), U2.2 (SW), U2.3 (SW), U2.4 (SW), U2.5 (SW)
- new net: C1.1, U2.6 (CBOOT)
- new net: C5.1, U2.7 (VCC)
- new net: D6.2 (A), R16.2
- new net: Q3.1 (G), R11.2
- new net: D3.2 (A), R19.2
- new net: Q6.1 (G), R14.2
- new net: J2.2 (Pin_2), Q2.2 (D)
- new net: R11.1, U3.7 (OUTA)
- new net DC_IN+: C5.2, FL1.1, J1.1 (Pin_1)
- new net DC_IN-: C5.1, FL1.2, J1.2 (Pin_2)
- new net DC_prefuse: C7.1, F1.2, FL1.4
- new net DC_preprot: D1.1 (A1), F1.1, NT1.2, NT2.2, Q1.5 (D), Q1.6 (D), Q1.7 (D), Q1.8 (D)
- new net adc_brightness: C16.1, RV3.2, U7.14 (PA0)
- new net button1: SW1.1 (A)
- new net button2: SW2.1 (A)
- new net indicator_led1: R16.1
- new net indicator_led2: R17.1
- new net indicator_led3: R18.1
- new net indicator_led4: R19.1
- new net lm73606_en: R10.1, U2.18 (EN)
- new net lm73606_pg: R1.1, U2.16 (PGOOD)
- new net tim15_ch1_ledstring5: U6.2 (INA), U7.35 (PB14)
- new net tim15_ch2_ledstring6: U6.4 (INB), U7.36 (PB15)
- new net tim3_ch1_ledstring1: U3.2 (INA), U7.22 (PA6)
- new net tim3_ch2_ledstring2: U3.4 (INB), U7.23 (PA7)
- new net tim3_ch3_ledstring3: U4.2 (INA), U7.26 (PB0)
- new net tim3_ch4_ledstring4: U4.4 (INB), U7.27 (PB1)
- new net vbat_meas: R8.2, U7.17 (PA3)
- no-connect marks 8 -> 2
Other:
- note added: "16V map to 3,2V"
- note added: "5A flow at about 16V"
- note removed: "11.8-14V norm."
- note removed: "Vled = 4.5V"
- moved on the sheet: C14, C15, RV1, RV2

Commit message: progress on schematic
Parts:
- removed C21: 22µF, Capacitor_THT:C_Radial_D5.0mm_H11.0mm_P2.00mm, symbol Waberinator_rev1-rescue:CP
- removed J1: 12VDC In, Connector_JST:JST_XH_B2B-XH-A_1x02_P2.50mm_Vertical, symbol Connector:Conn_01x02_Pin
- removed J11: Strang 0, symbol Connector:Conn_01x02_Male
- removed U5: LM75B, symbol Waberinator_rev1-rescue:LM75B
- added C11, C12, C27, C29, C31, C4, C6, C8: 100nF, Capacitor_SMD:C_0603_1608Metric_Pad1.08x0.95mm_HandSolder, symbol Device:C
- added C13: 22µF, Capacitor_SMD:C_1210_3225Metric_Pad1.33x2.70mm_HandSolder, symbol Device:C
- added C18: 47nF, Capacitor_SMD:C_0603_1608Metric_Pad1.08x0.95mm_HandSolder, symbol Device:C
- added C2, C26, C28, C30: 1µF, Capacitor_SMD:C_0603_1608Metric_Pad1.08x0.95mm_HandSolder, symbol Device:C
- added C20, C23: 10µF, Capacitor_SMD:C_1210_3225Metric_Pad1.33x2.70mm_HandSolder, symbol Device:C
- added C21, C22, C25: 56µF, Capacitor_SMD:C_Elec_5x5.8, symbol Device:C_Polarized
- added C24: 470nF, Capacitor_SMD:C_0603_1608Metric_Pad1.08x0.95mm_HandSolder, symbol Device:C
- added D7: BXFN-27G-21L-3C4-00-0-3, symbol Device:LED
- added FB1: FerriteBead, symbol Device:FerriteBead
- added J8: Conn_01x08_Pin, Connector_PinHeader_2.54mm:PinHeader_1x08_P2.54mm_Vertical, symbol Connector:Conn_01x08_Pin
- added J9: Conn_01x04_Pin, Connector_JST:JST_XH_B4B-XH-AM_1x04_P2.50mm_Vertical, symbol Connector:Conn_01x04_Pin
- added R20: 1, Resistor_SMD:R_0603_1608Metric_Pad0.98x0.95mm_HandSolder, symbol Device:R
- added R21: 100k, Resistor_SMD:R_0603_1608Metric_Pad0.98x0.95mm_HandSolder, symbol Device:R
- added R22, R23: 100, Resistor_SMD:R_0603_1608Metric_Pad0.98x0.95mm_HandSolder, symbol Device:R
- added U1: LM75B, Package_SO:SOIC-8_3.9x4.9mm_P1.27mm, symbol Sensor_Temperature:LM75B
- C1: value 479nF -> 470nF; footprint (none) -> Capacitor_SMD:C_0603_1608Metric_Pad1.08x0.95mm_HandSolder
- C14, C15, C16, C3, C9: footprint (none) -> Capacitor_SMD:C_0603_1608Metric_Pad1.08x0.95mm_HandSolder
- C5: SPR Digikey -> (none)
- C7: SPN 732-7672-1-ND -> (none); SPR Digikey -> (none); digikey (none) -> 732-7672-1-ND
- D1: SPN 732-9949-1-ND -> (none); SPR Digikey -> (none); digikey (none) -> 732-9949-1-ND
- D3, D4, D5, D6: footprint (none) -> LED_THT:LED_D3.0mm_Horizontal_O1.27mm_Z2.0mm
- FL1: SPN 240-2502-1-ND -> (none); digikey (none) -> 240-2502-1-ND
- J2, J3, J4, J5, J6, J7: footprint (none) -> Connector_JST:JST_XH_B2B-XH-AM_1x02_P2.50mm_Vertical; Digikey 609-3819-ND -> 455-B2B-XH-A-ND; MPN OQ0232510000G -> B2B-XH-A
- R1, R10, R11, R12, R13, R14, R15, R16, R17, R18, R19, R2, R3, R4, R5: footprint (none) -> Resistor_SMD:R_0603_1608Metric_Pad0.98x0.95mm_HandSolder
- RV1, RV2: footprint g7_hmi:potentiometer_P160 -> (none); Digikey (none) -> 987-1714-ND
- RV3: footprint g7_hmi:potentiometer_P160 -> (none)
- SW1: Digikey (none) -> EG5342-ND
Connections:
- net +3.3V is gone; now on net +3.3VA: RV1.1, RV2.1, RV3.1
- net indicator_led1 is gone; now on net tim1_ch1_indicator_led1: R16.1
- net indicator_led2 is gone; now on net tim1_ch2_indicator_led2: R17.1
- net indicator_led3 is gone; now on net tim1_ch3_indicator_led3: R18.1
- net indicator_led4 is gone; now on net tim1_ch4_indicator_led4: R19.1
- net +3V3: now also R1.2, U7.32 (VDD), U7.64 (VDD), C12.1, C13.1, C2.1, C4.1, C6.1, C8.1, FB1.1, J8.1 (Pin_1), R21.1, U1.8 (+Vs)
- net DC_IN+: now also J9.1 (Pin_1)
- net DC_IN-: now also J9.2 (Pin_2)
- net DC_prot: now also C18.1, C20.1, C21.1
- net RET: now also C11.2, C12.2, C13.2, C18.2, C2.2, C20.2, C21.2, C22.2, C23.2, C24.2, C25.2, C26.2, C27.2, C28.2, C29.2, C30.2, C31.2, C4.2, C6.2, C8.2, J8.3 (Pin_3), U1.4 (GND), U1.5 (A2), U1.6 (A1), U1.7 (A0)
- net VLed: now also C22.1, C23.1, C24.1, C25.1, C26.1, C27.1, C28.1, C29.1, C30.1, C31.1
- net button1: now also U7.29 (PB10)
- net button2: now also U7.30 (PB11)
- net lm73606_en: now also U7.38 (PC7)
- net lm73606_pg: now also U7.39 (PC8)
- net ledstring3_drv_en: now reaches U4.1 (ENA)
- net ledstring3_drv_en: now also U7.10 (PC2)
- net ledstring4_drv_en: now reaches U4.8 (ENB)
- net ledstring4_drv_en: now also U7.11 (PC3)
- net +3.3VA: now reaches U7.13 (VDDA)
- net +3.3VA: now also C11.1, FB1.2
- net spi1_sck: now reaches U7.21 (PA5)
- net ledstring5_drv_en: now reaches U7.24 (PC4)
- net ledstring5_drv_en: now also U6.1 (ENA)
- net ledstring6_drv_en: now reaches U7.25 (PC5)
- net ledstring6_drv_en: now also U6.8 (ENB)
- net lm75b_int: now reaches U7.37 (PC6)
- net lm75b_int: now also U1.3 (O.S.)
- net tim1_ch1_indicator_led1: now reaches U7.41 (PA8)
- net tim1_ch2_indicator_led2: now reaches U7.42 (PA9)
- net tim1_ch3_indicator_led3: now reaches U7.43 (PA10)
- net tim1_ch4_indicator_led4: now reaches U7.44 (PA11)
- net swd_tms: now reaches U7.46 (PA13)
- net swd_tms: now also J8.4 (Pin_4)
- net swd_tck: now reaches U7.49 (PA14)
- net swd_tck: now also J8.2 (Pin_2)
- net swd_swo: now reaches U7.55 (PB3)
- net swd_swo: now also J8.6 (Pin_6)
- net spi1_miso: now reaches U7.56 (PB4)
- net spi1_mosi: now reaches U7.57 (PB5)
- net usart1_tx_mcu: now reaches U7.58 (PB6)
- net usart1_tx_mcu: now also J8.8 (Pin_8), R23.2
- net usart1_rx_mcu: now reaches U7.59 (PB7)
- net usart1_rx_mcu: now also J8.7 (Pin_7), R22.2
- net i2c1_scl: now reaches U7.61 (PB8)
- net i2c1_scl: now also U1.2 (SCL)
- net i2c1_sda: now reaches U7.62 (PB9)
- net i2c1_sda: now also U1.1 (SDA)
- net ~{rst}: now reaches U7.7 (NRST)
- net ~{rst}: now also J8.5 (Pin_5), R21.2
- net ledstring1_drv_en: now reaches U7.8 (PC0)
- net ledstring1_drv_en: now also U3.1 (ENA)
- net ledstring2_drv_en: now reaches U7.9 (PC1)
- net ledstring2_drv_en: now also U3.8 (ENB)
- new net: D7.1 (K), R20.1
- new net: J9.3 (Pin_3), R22.1
- new net: J9.4 (Pin_4), R23.1
Other:
- note added: "Representative for the Light Boards - 60 Boards in total - 3 LEDs, 1 Resistor each - 180 LEDs, 60 Resistors total"
- note added: "Teilenummern für vorkonfektionierte Kab"
- note added: "alternate pins?"
- note removed: "Temp. SMPS"
- moved on the sheet: C14, C15, C16, J2, J3, J4, J5, J6, J7, Q2, Q3, Q4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
